File: WVM.kicad_sch (KiCad schematic)
At the start: 7 parts, among them J1 USB4215-03-A_REVA, U1 IIS3DWBTR, U2 MCP9808_DFN, U3 CH340C, U4 TPS63036YFGT, U5 NORA-W106-00B, U6 TP4056-42-ESOP8

Commit message: Modified Schematic 07.10.25
Parts:
- removed J1: USB4215-03-A_REVA, USB4215-03-A:USB4215-03-A_REVA, symbol USB4215-03-A_REVA:USB4215-03-A_REVA
- removed U1: IIS3DWBTR, IIS3DWBTR:LGA-14L_2P5X3X0P83_STM, symbol IIS3DWBTR:IIS3DWBTR
- removed U2: MCP9808_DFN, Package_DFN_QFN:DFN-8-1EP_3x2mm_P0.5mm_EP1.7x1.4mm, symbol Sensor_Temperature:MCP9808_DFN
- removed U3: CH340C, Package_SO:SOIC-16_3.9x9.9mm_P1.27mm, symbol Interface_USB:CH340C
- removed U4: TPS63036YFGT, TPS63036YFGT:TPS63036YFGT, symbol TPS63036YFGT:TPS63036YFGT
- removed U5: NORA-W106-00B, NORA-W106-00B:XCVR_NORA-W106-00B, symbol NORA-W106-00B:NORA-W106-00B
- removed U6: TP4056-42-ESOP8, Package_SO:SOIC-8-1EP_3.9x4.9mm_P1.27mm_EP2.41x3.3mm_ThermalVias, symbol Battery_Management:TP4056-42-ESOP8
- added C1, C2, C3: 10uF, symbol Device:C
- added C4: 30uF, symbol Device:C
- added C5, C6: 0.1uF, symbol Device:C
- added C7, C8: 0.1Uf, symbol Device:C
- added D1, D2: LED, symbol Device:LED
- added D3, D4: D, symbol Device:D
- added J1: Conn_01x02_Pin, daFootprintsBX:JST_S2B-PH-SM4-TB, symbol Connector:Conn_01x02_Pin
- added J3: USB4215-03-A_REVA, USB4215-03-A:USB4215-03-A_REVA, symbol USB4215-03-A_REVA:USB4215-03-A_REVA
- added L1: 1.5uH, symbol Device:L
- added Q1: 2SK3019, Package_TO_SOT_SMD:SOT-523, symbol Transistor_FET:2SK3019
- added R1, R2: 1k, symbol Device:R
- added R3: 2k, symbol Device:R
- added R4: 287k, symbol Device:R
- added R5: 51.1k, symbol Device:R
- added U1: CH340C, Package_SO:SOIC-16_3.9x9.9mm_P1.27mm, symbol Interface_USB:CH340C
- added U2: TP4056-42-ESOP8, Package_SO:SOIC-8-1EP_3.9x4.9mm_P1.27mm_EP2.41x3.3mm_ThermalVias, symbol Battery_Management:TP4056-42-ESOP8
- added U3: IIS3DWBTR, LGA-14L_2P5X3X0P83_STM, symbol IIS3DWBTR:IIS3DWBTR
- added U5: MCP9808_DFN, Package_DFN_QFN:DFN-8-1EP_3x2mm_P0.5mm_EP1.7x1.4mm, symbol Sensor_Temperature:MCP9808_DFN
- added U6: TPS63036YFGT, TPS63036YFGT:TPS63036YFGT, symbol TPS63036YFGT:TPS63036YFGT
- added U7: NORA-W106-00B, NORA-W106-00B:XCVR_NORA-W106-00B, symbol NORA-W106-00B:NORA-W106-00B
Connections:
- net D+: now also J3.A6 (DP1), U1.5 (UD+)
- net D-: now also J3.A7 (DN1), U1.6 (UD-)
- new net: Q1.3 (D), U1.3 (RXD)
- new net: C3.2, C4.2, R5.2, U6.B2 (PS/SYNC), U6.C2 (GND)
- new net: R3.1, U2.2 (PROG)
- new net: R1.1, U2.6 (~{STDBY})
- new net: R2.2, U2.7 (~{CHRG})
- new net: D2.1 (K), R1.2
- new net: D4.1 (K), U1.14 (~{RTS})
- new net: C6.2, U1.4 (V3)
- new net: D3.1 (K), U1.2 (TXD)
- new net: L1.1, U6.B1 (L1)
- new net: L1.2, U6.C1 (L2)
- new net: R4.2, R5.1, U6.D2 (FB)
- new net: D1.1 (K), R2.1
- new net 3V3: C4.1, C7.2, C8.1, Q1.1 (G), R4.1, U3.5 (VDD_IO), U3.8 (VDD), U5.8 (V_{DD}), U6.D1 (VOUT), U7.A7 (VCCIO), U7.A8 (VCC)
- new net 5V: C2.1, C3.1, J1.1 (Pin_1), U2.5 (BAT), U6.A1 (VIN), U6.A2 (EN)
- new net BOOT: D4.2 (A), U7.F7 (GPIO0/BOOT)
- new net CLK: U3.13 (SPC/SCL)
- new net CS: U3.12 (CS)
- new net GND: C1.2, C2.2, C5.1, C6.1, C7.1, C8.2, J1.2 (Pin_2), J3.A1_B12 (GND_A), J3.SH1 (SHIELD), R3.2, U1.1 (GND), U2.1 (TEMP), U2.3 (GND), U2.9 (EPAD), U3.2 (RES), U3.3 (RES), U3.6 (GND), U3.7 (GND), U5.4 (GND), U5.9 (EP/GND), U7.A1 (EGP), U7.A9 (EGP__1), U7.B2 (EGP__2), U7.B8 (EGP__3), U7.E4 (EGP__4), U7.E5 (EGP__5), U7.F4 (EGP__6), U7.F5 (EGP__7), U7.K2 (EGP__8), U7.K3 (EGP__9), U7.K5 (EGP__10), U7.K7 (EGP__11), U7.K8 (EGP__12), U7.L1 (EAGP), U7.L9 (EAGP__1), U7.M1 (EAGP__2), U7.M2 (EAGP__3), U7.M8 (EAGP__4), U7.M9 (EAGP__5)
- new net INT: U3.4 (INT1), U7.E8 (GPIO1)
- new net MISO: U3.1 (SDO/SA0)
- new net MOSI: U3.14 (SDI/SDO/SDA)
- new net RXD: Q1.2 (S), U7.G8 (U0TXD/GPIO43)
- new net SCL: U5.2 (SCL)
- new net SDA: U5.1 (SDA)
- new net TXD: D3.2 (A), U7.G9 (U0RXD/GPIO44)
- new net VCC: C1.1, C5.2, D1.2 (A), D2.2 (A), J3.A4_B9 (VBUS_A), U1.16 (VCC), U2.4 (V_{CC}), U2.8 (CE)
- no-connect marks 5 -> 53
Other:
- note added: "Buck/Boost Converter"
- note added: "Power Supply 5V"

Commit message: message
Parts:
- added C10, C9: 0.1uF 50V 10%, Capacitor_SMD:C_01005_0402Metric, symbol Device:C
- added SW1, SW3: SW_Push, Button_Switch_SMD:SW_Push_1P1T_NO_E-Switch_TL3301NxxxxxG, symbol Switch:SW_Push
- C1, C2, C3, C4, C5, C6, C7, C8: footprint (none) -> Capacitor_SMD:C_01005_0402Metric
- D1, D2: footprint (none) -> LED_SMD:LED_0402_1005Metric
- D3, D4: footprint (none) -> Diode_SMD:D_0402_1005Metric
- L1: footprint (none) -> Inductor_SMD:L_0402_1005Metric
- R1, R2, R3, R4, R5: footprint (none) -> Resistor_SMD:R_0402_1005Metric
- U3: footprint LGA-14L_2P5X3X0P83_STM -> IIS3DWBTR:LGA-14L_2P5X3X0P83_STM
Connections:
- net 3V3: no longer U3.5 (VDD_IO), U7.A7 (VCCIO)
- net CLK: now also U7.B1 (FSPICLK/GPIO36)
- net CS: now also U7.B3 (FSPICS0/GPIO34)
- net GND: now also C10.1, C9.1, SW1.1, SW3.1; no longer U3.2 (RES), U3.3 (RES), U3.6 (GND)
- net MISO: now also U7.C1 (FSPIQ/GPIO37)
- net MOSI: now also U7.C2 (FSPID/GPIO35)
- net SCL: now also U7.A2 (FSPIWP/GPIO38)
- net SDA: now also U7.D3 (FSPIHD/GPIO33)
- net RESET: now reaches U7.J3 (~{RESET})
- net RESET: now also C9.2, SW1.2
- net INT: no longer names the net of U3.4 (INT1)
- net INT: no longer U7.E8 (GPIO1)
- new net GPIO1: C10.2, SW3.2, U7.E8 (GPIO1)
- new net VCC_IO: U3.5 (VDD_IO), U7.A7 (VCCIO)
- no-connect marks 53 -> 55
Other:
- note added: "NORA-W106-00B-MC"
- note added: "TEMPERATURE SENSOR"
- note added: "USB TO UART"
- note added: "VIBRATION SENSOR"
- moved on the sheet: C8, U7

Commit message: cleaned schematic
Parts:
- removed C1, C2: 10uF, Capacitor_SMD:C_01005_0402Metric, symbol Device:C
- removed D1, D2: LED, LED_SMD:LED_0402_1005Metric, symbol Device:LED
- removed J1: Conn_01x02_Pin, daFootprintsBX:JST_S2B-PH-SM4-TB, symbol Connector:Conn_01x02_Pin
- removed J3: USB4215-03-A_REVA, USB4215-03-A:USB4215-03-A_REVA, symbol USB4215-03-A_REVA:USB4215-03-A_REVA
- removed L1: 1.5uH, Inductor_SMD:L_0402_1005Metric, symbol Device:L
- removed R1, R2: 1k, Resistor_SMD:R_0402_1005Metric, symbol Device:R
- removed R3: 2k, Resistor_SMD:R_0402_1005Metric, symbol Device:R
- removed U2: TP4056-42-ESOP8, Package_SO:SOIC-8-1EP_3.9x4.9mm_P1.27mm_EP2.41x3.3mm_ThermalVias, symbol Battery_Management:TP4056-42-ESOP8
- removed U6: TPS63036YFGT, TPS63036YFGT:TPS63036YFGT, symbol TPS63036YFGT:TPS63036YFGT
- added C11: 10uF, Capacitor_SMD:C_01005_0402Metric, symbol Device:C
- added C12: 30uF, Capacitor_SMD:C_01005_0402Metric, symbol Device:C
- added D5, D6: LED, LED_SMD:LED_0402_1005Metric, symbol Device:LED
- added J2: USB4215-03-A_REVA, USB4215-03-A:USB4215-03-A_REVA, symbol USB4215-03-A_REVA:USB4215-03-A_REVA
- added L2: 1.5uH, Inductor_SMD:L_0402_1005Metric, symbol Device:L
- added R6: 287k, Resistor_SMD:R_0402_1005Metric, symbol Device:R
- added R7: 51.1k, Resistor_SMD:R_0402_1005Metric, symbol Device:R
- added R8: 2k, Resistor_SMD:R_0402_1005Metric, symbol Device:R
- added U4: TPS63036YFGT, TPS63036YFGT:TPS63036YFGT, symbol TPS63036YFGT:TPS63036YFGT
- added U6: TP4056-42-ESOP8, Package_SO:SOIC-8-1EP_3.9x4.9mm_P1.27mm_EP2.41x3.3mm_ThermalVias, symbol Battery_Management:TP4056-42-ESOP8
- C4: value 30uF -> 10uF
- R4: value 287k -> 1k
- R5: value 51.1k -> 1k
Connections:
- net 3V3: now also C12.1, R6.1, U4.D1 (VOUT); no longer C4.1, R4.1
- net D+: now also J2.A6 (DP1)
- net D-: now also J2.A7 (DN1)
- net GND: now also C3.2, C4.2, C11.2, C12.2, J2.A1_B12 (GND_A), J2.SH1 (SHIELD), R7.2, R8.2, U4.B2 (PS/SYNC), U4.C2 (GND), U6.1 (TEMP), U6.3 (GND), U6.9 (EPAD)
- net at R5.1: now also D6.1 (K); no longer R4.2
- net 5V: no longer names the net of C3.1
- net 5V: now also D5.2 (A), D6.2 (A), J2.A4_B9 (VBUS_A), U6.4 (V_{CC})
- new net: L2.1, U4.B1 (L1)
- new net: L2.2, U4.C1 (L2)
- new net: D5.1 (K), R4.1
- new net: R6.2, R7.1, U4.D2 (FB)
- new net: R8.1, U6.2 (PROG)
- new net: R5.2, U6.6 (~{STDBY})
- new net: R4.2, U6.7 (~{CHRG})
- new net +BAT: C11.1, C4.1, U4.A1 (VIN), U4.A2 (EN), U6.5 (BAT)
Other:
- note added: "3.3V Buck Boost Converter"
- note added: "Charging Module"
- note removed: "Buck/Boost Converter"
- note removed: "Power Supply 5V"
- moved on the sheet: C10, C5, C6, C7, C8, C9, D3, D4, Q1, SW1, SW3, U1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

Commit message: Completed schematic 09.10.25
Parts:
- removed C10: 0.1uF 50V 10%, Capacitor_SMD:C_01005_0402Metric, symbol Device:C
- removed C7, C8: 0.1Uf, Capacitor_SMD:C_01005_0402Metric, symbol Device:C
- removed D3, D4: D, Diode_SMD:D_0402_1005Metric, symbol Device:D
- removed Q1: 2SK3019, Package_TO_SOT_SMD:SOT-523, symbol Transistor_FET:2SK3019
- removed SW1, SW3: SW_Push, Button_Switch_SMD:SW_Push_1P1T_NO_E-Switch_TL3301NxxxxxG, symbol Switch:SW_Push
- removed U1: CH340C, Package_SO:SOIC-16_3.9x9.9mm_P1.27mm, symbol Interface_USB:CH340C
- removed U5: MCP9808_DFN, Package_DFN_QFN:DFN-8-1EP_3x2mm_P0.5mm_EP1.7x1.4mm, symbol Sensor_Temperature:MCP9808_DFN
- removed U7: NORA-W106-00B, NORA-W106-00B:XCVR_NORA-W106-00B, symbol NORA-W106-00B:NORA-W106-00B
- added C1, C2, C3, C4: 0.1uF, Capacitor_SMD:C_0402_1005Metric, symbol Device:C
- added P1: S2B-PH-SM4-TB, S2B_PH_SM4_TB:JST_S2B-PH-SM4-TB, symbol S2B-PH-SM4-TB:S2B-PH-SM4-TB
- added Q1, Q2: BSS138, Package_TO_SOT_SMD:SOT-23, symbol Transistor_FET:BSS138
- added SW1, SW2: SW_SPST, Button_Switch_SMD:SW_SPST_B3U-1000P, symbol Switch:SW_SPST
- added U1: NORA-W106-00B, NORA-W106-00B:XCVR_NORA-W106-00B, symbol NORA-W106-00B:NORA-W106-00B
- added U2: CH340C, Package_SO:SOIC-16_3.9x9.9mm_P1.27mm, symbol Interface_USB:CH340C
- added U6: MCP9808_DFN, Package_DFN_QFN:DFN-8-1EP_3x2mm_P0.5mm_EP1.7x1.4mm, symbol Sensor_Temperature:MCP9808_DFN
- C10: renamed from C4; footprint Capacitor_SMD:C_01005_0402Metric -> Capacitor_SMD:C_0402_1005Metric
- C11: renamed from C12; footprint Capacitor_SMD:C_01005_0402Metric -> Capacitor_SMD:C_0402_1005Metric
- C5: footprint Capacitor_SMD:C_01005_0402Metric -> Capacitor_SMD:C_0402_1005Metric
- C6: value 0.1uF -> 1uF; footprint Capacitor_SMD:C_01005_0402Metric -> Capacitor_SMD:C_0402_1005Metric
- C7: renamed from C3; footprint Capacitor_SMD:C_01005_0402Metric -> Capacitor_SMD:C_0402_1005Metric
- C8: renamed from C11; footprint Capacitor_SMD:C_01005_0402Metric -> Capacitor_SMD:C_0402_1005Metric
- C9: value 0.1uF 50V 10% -> 0.1uF; footprint Capacitor_SMD:C_01005_0402Metric -> Capacitor_SMD:C_0402_1005Metric
- renumbered D6 to D1, D5 to D2, J2 to J1, L2 to L1, R5 to R1, R4 to R2, R8 to R3, R6 to R4, R7 to R5, U6 to U5
Connections:
- net VCC is gone; now on net GND: C5.2
- net VCC_IO is gone; now on net 3V3: U3.5 (VDD_IO)
- net +BAT: now also P1.1
- net 3V3: now also C5.1, C9.2, C1.1, C2.1, U1.A7 (VCCIO), U1.A8 (VCC), U2.16 (VCC), U2.4 (V3), U6.8 (V_{DD})
- net BOOT: now also Q2.3 (D), U1.F7 (GPIO0/BOOT)
- net CLK: now also U1.B1 (FSPICLK/GPIO36)
- net CS: now also U1.B3 (FSPICS0/GPIO34)
- net D+: now also U2.5 (UD+)
- net D-: now also U2.6 (UD-)
- net GND: now also C6.2, U3.2 (RES), U3.3 (RES), U3.6 (GND), C1.2, C2.2, C3.1, C4.1, SW1.1 (A), SW2.1 (A), U1.A1 (EGP), U1.A9 (EGP__1), U1.B2 (EGP__2), U1.B8 (EGP__3), U1.E4 (EGP__4), U1.E5 (EGP__5), U1.F4 (EGP__6), U1.F5 (EGP__7), U1.K2 (EGP__8), U1.K3 (EGP__9), U1.K5 (EGP__10), U1.K7 (EGP__11), U1.K8 (EGP__12), U1.L1 (EAGP), U1.L9 (EAGP__1), U1.M1 (EAGP__2), U1.M2 (EAGP__3), U1.M8 (EAGP__4), U1.M9 (EAGP__5), U2.1 (GND), U6.4 (GND), U6.5 (A2), U6.6 (A1), U6.7 (A0), U6.9 (EP/GND); no longer C5.1, C6.1
- net GPIO1: now also C4.2, SW2.2 (B), U1.E8 (GPIO1)
- net MISO: now also U1.C1 (FSPIQ/GPIO37)
- net MOSI: now also U1.C2 (FSPID/GPIO35)
- net RESET: now also C3.2, SW1.2 (B), U1.J3 (~{RESET}); no longer C9.2
- net SCL: now also U1.A2 (FSPIWP/GPIO38), U6.2 (SCL)
- net SDA: now also U1.D3 (FSPIHD/GPIO33), U6.1 (SDA)
- net INT1: now reaches U3.4 (INT1)
- net INT2: now reaches U3.9 (INT2)
- new net: Q1.1 (G), Q2.2 (S), U2.13 (~{DTR})
- new net: Q1.2 (S), Q2.1 (G), U2.14 (~{RTS})
- new net -BAT: P1.2
- new net EN: C6.1, Q1.3 (D)
- new net RX: U1.G9 (U0RXD/GPIO44), U2.2 (TXD)
- new net TX: U1.G8 (U0TXD/GPIO43), U2.3 (RXD)
- no-connect marks 55 -> 46
Other:
- note added: "Temperature Sensor"
- note added: "USB to UART Bridge"
- note added: "Vibration Sensor"
- note removed: "NORA-W106-00B-MC"
- note removed: "TEMPERATURE SENSOR"
- note removed: "USB TO UART"
- note removed: "VIBRATION SENSOR"
- moved on the sheet: C10, C11, C7, C8, D1, D2, J1, L1, R1, R2, R3, R4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

Commit message: 09/08/2025
Parts:
- added H1, H2, H3, H4: MountingHole, MountingHole:MountingHole_2.2mm_M2, symbol Mechanical:MountingHole
Other:
- note added: "BOOT BUTTON"
- note added: "NORA-W106-00B"
- note added: "RESET BUTTON"
- moved on the sheet: C1, P1, U1

Commit message: 10-10-2025
Parts:
- removed L1: 1.5uH, Inductor_SMD:L_0402_1005Metric, symbol Device:L
- added L1: LPS3015-152MLC, LPS3015-152MLC:IND_LPS3015-152MLC, symbol LPS3015-152MLC:LPS3015-152MLC
Connections:
- net at U4.B1 (L1): now also L1.1
- net at U4.C1 (L2): now also L1.2
- no-connect marks 46 -> 47
Changed lines of the file:
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@@
+	)
+	(no_connect
+		(at 224.79 83.82)
 	)
 	(no_connect
@@
 	(wire
 		(pts
+			(xy 248.92 55.88) (xy 248.92 60.96)
+		)
+		(stroke
+			(width 0)
+			(type default)
+		)
+	)
+	(wire
+		(pts
 			(xy 88.9 148.59) (xy 91.44 148.59)
 		)
@@
 	(wire
 		(pts
+			(xy 223.52 55.88) (xy 233.68 55.88)
+		)
+		(stroke
+			(width 0)
+			(type default)
+		)
+	)
+	(wire
+		(pts
 			(xy 88.9 140.97) (xy 91.44 140.97)
 		)
@@
 	(wire
 		(pts
+			(xy 223.52 60.96) (xy 223.52 55.88)
+		)
+		(stroke
+			(width 0)
+			(type default)
+		)
+	)
+	(wire
+		(pts
 			(xy 190.5 85.09) (xy 193.04 85.09)
 		)
@@
 		(pts
 			(xy 177.8 138.43) (xy 177.8 140.97)
+		)
+		(stroke
+			(width 0)
+			(type default)
+		)
+	)
+	(wire
+		(pts
+			(xy 241.3 55.88) (xy 248.92 55.88)
 		)
 		(stroke
@@
 				(justify right)
 				(hide yes)
+			)
+		)
+	)
+	(symbol
+		(lib_id "LPS3015-152MLC:LPS3015-152MLC")
+		(at 236.22 60.96 0)
+		(unit 1)
+		(exclude_from_sim no)
+		(in_bom yes)
+		(on_board yes)
+		(dnp no)
+		(fields_autoplaced yes)
+		(property "Reference" "L1"
+			(at 236.22 54.61 0)
+			(effects
+				(font
+					(size 1.27 1.27)
+				)
+			)
+		)
+		(property "Value" "LPS3015-152MLC"
+			(at 236.22 57.15 0)
+			(effects
+				(font
+					(size 1.27 1.27)
+				)
+			)
+		)
+		(property "Footprint" "LPS3015-152MLC:IND_LPS3015-152MLC"
+			(at 236.22 60.96 0)
+			(effects
+				(font
+					(size 1.27 1.27)
+				)
+				(justify bottom)
+				(hide yes)
+			)
+		)
+		(property "Datasheet" ""
+			(at 236.22 60.96 0)
+			(effects
+				(font
+					(size 1.27 1.27)
+				)
+				(hide yes)
+			)
+		)
+		(property "Description" ""
+			(at 236.22 60.96 0)
+			(effects
+				(font
+					(size 1.27 1.27)
+				)
+				(hide yes)
+			)
+		)
+		(property "MF" "Coilcraft"
+			(at 236.22 60.96 0)
+			(effects
+				(font
+					(size 1.27 1.27)
+				)
+				(justify bottom)
+				(hide yes)
+			)
+		)
+		(property "MAXIMUM_PACKAGE_HEIGHT" "1.5mm"
+			(at 236.22 60.96 0)
+			(effects
+				(font
+					(size 1.27 1.27)
+				)
+				(justify bottom)
+				(hide yes)
+			)
+		)
+		(property "Package" "None"
+			(at 236.22 60.96 0)
+			(effects
+				(font
+					(size 1.27 1.27)
+				)
+				(justify bottom)
+				(hide yes)
+			)
+		)
+		(property "Price" "None"
+			(at 236.22 60.96 0)
+			(effects
+				(font
+					(size 1.27 1.27)
+				)
+				(justify bottom)
+				(hide yes)
+			)
+		)
+		(property "Check_prices" "https://www.snapeda.com/parts/LPS3015-152MLC/Coilcraft/view-part/?ref=eda"
+			(at 236.22 60.96 0)
+			(effects
+				(font
+					(size 1.27 1.27)
+				)
+				(justify bottom)
+				(hide yes)
+			)
+		)
+		(property "STANDARD" "Manufacturer Recommendations"
+			(at 236.22 60.96 0)
+			(effects
+				(font
+					(size 1.27 1.27)
+				)
+				(justify bottom)
+				(hide yes)
+			)
+		)
+		(property "PARTREV" "12/13/21"
+			(at 236.22 60.96 0)
+			(effects
+				(font
+					(size 1.27 1.27)
+				)
+				(justify bottom)
+				(hide yes)
+			)
+		)
+		(property "SnapEDA_Link" "https://www.snapeda.com/parts/LPS3015-152MLC/Coilcraft/view-part/?ref=snap"
+			(at 236.22 60.96 0)
+			(effects
+				(font
+					(size 1.27 1.27)
+				)
+				(justify bottom)
+				(hide yes)
+			)
+		)
+		(property "MP" "LPS3015-152MLC"
+			(at 236.22 60.96 0)
+			(effects
+				(font
+					(size 1.27 1.27)
+				)
+				(justify bottom)
+				(hide yes)
+			)
+		)
+		(property "Description_1" "Power inductor, shielded, 20% tol, SMT, RoHS"
+			(at 236.22 60.96 0)
+			(effects
+				(font
+					(size 1.27 1.27)
+				)
+				(justify bottom)
+				(hide yes)
+			)
+		)
+		(property "Availability" "In Stock"
+			(at 236.22 60.96 0)
+			(effects
+				(font
+					(size 1.27 1.27)
+				)
+				(justify bottom)
+				(hide yes)
+			)
+		)
+		(property "MANUFACTURER" "Coilcraft"
+			(at 236.22 60.96 0)
+			(effects
+				(font
+					(size 1.27 1.27)
+				)
+				(justify bottom)
+				(hide yes)
+			)
+		)
+		(pin "1"
+		)
+		(pin "2"
+		)
+		(instances
+			(project ""
+				(path "/5968613b-5d72-4cb2-8e74-d6867cb32824"
+					(reference "L1")
+					(unit 1)
+				)
 			)
 		)
@@
 					(unit 1)
 				)
-			)
-		)
-	)
-	(symbol
-		(lib_id "Device:L")
-		(at 237.49 55.88 90)
-		(unit 1)
-		(exclude_from_sim no)
-		(in_bom yes)
-		(on_board yes)
-		(dnp no)
-		(property "Reference" "L1"
-			(at 237.49 53.848 90)
-			(effects
-				(font
-					(size 1.27 1.27)
-				)
-			)
-		)
-		(property "Value" "1.5uH"
-			(at 237.49 57.404 90)
-			(effects
-				(font
-					(size 1.27 1.27)
-				)
-			)
-		)
-		(property "Footprint" "Inductor_SMD:L_0402_1005Metric"
-			(at 237.49 55.88 0)
-			(effects
-				(font
-					(size 1.27 1.27)
-				)
-				(hide yes)
-			)
-		)
-		(property "Datasheet" "~"
-			(at 237.49 55.88 0)
-			(effects
-				(font
-					(size 1.27 1.27)
-				)
-				(hide yes)
-			)
-		)
-		(property "Description" "Inductor"
-			(at 237.49 55.88 0)
-			(effects
-				(font
-					(size 1.27 1.27)
-				)
-				(hide yes)
-			)
-		)
-		(pin "2"
-		)
-		(pin "1"
-		)
-		(instances
-			(project "WVM"
-				(path "/5968613b-5d72-4cb2-8e74-d6867cb32824"
-					(reference "L1")
-					(unit 1)
-				)
