File: WVM.kicad_sch (KiCad schematic)
At the start: 35 parts, among them J1 USB4215-03-A_REVA, J2 Conn_01x02_Pin, Q1 BSS138, Q2 BSS138, SW1 SW_SPST, SW2 SW_SPST, U1 NORA-W106-00B, U2 CH340C, U3 IIS3DWBTR, U4 TPS63036YFGT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

Commit message: 17102025
Parts:
- removed C2, C9: 0.1uF, Capacitor_SMD:C_0402_1005Metric, symbol Device:C
- removed C6: 1uF, Capacitor_SMD:C_0402_1005Metric, symbol Device:C
- removed Q1, Q2: BSS138, Package_TO_SOT_SMD:SOT-23, symbol Transistor_FET:BSS138
- removed U2: CH340C, Package_SO:SOIC-16_3.9x9.9mm_P1.27mm, symbol Interface_USB:CH340C
- removed U6: MCP9808_DFN, Package_DFN_QFN:DFN-8-1EP_3x2mm_P0.5mm_EP1.7x1.4mm, symbol Sensor_Temperature:MCP9808_DFN
- added J4, J5, J6: Conn_01x02_Pin, Connector_PinHeader_1.00mm:PinHeader_1x02_P1.00mm_Vertical, symbol Connector:Conn_01x02_Pin
Connections:
- net -BAT is gone; now on net GND: J2.2 (Pin_2)
- net 3V3: now also J4.1 (Pin_1)
- net BOOT: now also J6.2 (Pin_2)
- net EN: now also U1.H8 (GPIO2), J6.1 (Pin_1)
- net GND: now also J4.2 (Pin_2)
- net INT1: now also U1.H9 (GPIO8)
- net INT2: now also U1.E7 (GPIO9)
- net RX: now also J5.1 (Pin_1)
- net TX: now also J5.2 (Pin_2)
- net D+: no longer names the net of J1.A6 (DP1)
- net D-: no longer names the net of J1.A7 (DN1)
- net SCL: no longer names the net of U1.A2 (FSPIWP/GPIO38)
- net SDA: no longer names the net of U1.D3 (FSPIHD/GPIO33)
- no-connect marks 47 -> 42
Other:
- note removed: "Temperature Sensor"
- note removed: "USB to UART Bridge"
- moved on the sheet: C10, C11, C3, C4, C5, C7, C8, D1, D2, H1, H2, H3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
